Commit message: add joint_limited urdf of fetch. current fetch.urdf is joint_limited version

File: fetch_description/robots/calibrated_2016_02_03_18_18_34.urdf (robot description, URDF)
Before this commit: robot fetch, 26 links, 25 joints
Joints:
- joint forearm_roll_joint: limit lower=-2.0 upper=2.0 effort=29.35 velocity=1.571 -> effort=29.35 velocity=1.571; type revolute -> continuous
- joint torso_lift_joint: limit lower=0 upper=0.1 effort=450.0 velocity=0.1 -> lower=0 upper=0.4 effort=450.0 velocity=0.1
- joint upperarm_roll_joint: limit lower=-2.0 upper=2.0 effort=76.94 velocity=1.571 -> effort=76.94 velocity=1.571; type revolute -> continuous
- joint wrist_roll_joint: limit lower=-2.0 upper=2.0 effort=7.36 velocity=2.268 -> effort=7.36 velocity=2.268; type revolute -> continuous

File: fetch_description/robots/calibrated_2016_02_03_18_18_34_joint_limited.urdf (robot description, URDF)
Before this commit: robot fetch, 26 links, 25 joints
Joints:
- joint torso_lift_joint: limit lower=0 upper=0.1 effort=450.0 velocity=0.1 -> lower=0 upper=0.4 effort=450.0 velocity=0.1
